File: PCB/eggkeeb.kicad_sch (KiCad schematic)
At the start: 130 parts, among them SW1 SW_Push, SW10 SW_Push, SW11 SW_Push, SW12 SW_Push, SW13 SW_Push, SW14 SW_Push, SW15 SW_Push, SW16 SW_Push, SW17 SW_Push, SW18 SW_Push, SW19 SW_Push, SW2 SW_Push, SW20 SW_Push, SW21 SW_Push, SW22 SW_Push, SW23 SW_Push, SW24 SW_Push, SW25 SW_Push, SW26 SW_Push, SW27 SW_Push, SW28 SW_Push, SW29 SW_Push, SW3 SW_Push, SW30 SW_Push, SW31 SW_Push, SW32 SW_Push, SW33 SW_Push, SW34 SW_Push, SW35 SW_Push, SW36 SW_Push, SW37 SW_Push, SW38 SW_Push, SW39 SW_Push, SW4 SW_Push, SW40 SW_Push, SW41 SW_Push, SW42 SW_Push, SW43 SW_Push, SW44 SW_Push, SW45 SW_Push, SW46 SW_Push, SW47 SW_Push, SW48 SW_Push, SW49 SW_Push, SW5 SW_Push, SW50 SW_Push, SW51 SW_Push, SW52 SW_Push, SW53 SW_Push, SW54 SW_Push, SW55 SW_Push, SW56 SW_Push, SW57 SW_Push, SW58 SW_Push, SW59 SW_Push, SW6 SW_Push, SW60 SW_Push, SW61 SW_Push, SW62 SW_Push, SW63 SW_Push, SW65 SW_Push, SW7 SW_Push, SW8 SW_Push, SW9 SW_Push

Commit message: Add files via upload
Parts:
- added D62, D63, D64, D65, D66, D67, D68, D69, D70, D71, D72, D73, D77, D78, D79, D80, D81, D82, D83, D84, D85, D86, D87: 1N4148, Diode_THT:D_DO-35_SOD27_P7.62mm_Horizontal, symbol Diode:1N4148
- added S2, S3, S4, S5: MX_stab, PCM_marbastlib-mx:STAB_MX_2.25u, symbol PCM_marbastlib-mx:MX_stab
- added SW16: RotaryEncoder_Switch, symbol Device:RotaryEncoder_Switch
- added SW63, SW64, SW65, SW66, SW67, SW68, SW69, SW70, SW71, SW72, SW73, SW74, SW78, SW79, SW80, SW81, SW82, SW83, SW84, SW85, SW86, SW87, SW88: SW_Push, symbol Switch:SW_Push
- added U1: ER_OLEDM0.91_1x-I2C, Display:ER_OLEDM0.91_1x-I2C, symbol Display_Graphic:ER_OLEDM0.91_1x-I2C
- S1: footprint PCM_marbastlib-mx:STAB_MX_P_6.25u -> PCM_marbastlib-mx:STAB_MX_2u
- renumbered D20 to D1, D29 to D10, D30 to D11, D31 to D12, D32 to D13, D33 to D14, D34 to D15, D1 to D16, D6 to D17, D7 to D18, D8 to D19, D21 to D2, D9 to D20, D10 to D21, D11 to D22, D12 to D23, D13 to D24, D14 to D25, D15 to D26, D16 to D27, D17 to D28, D18 to D29, D22 to D3, D19 to D30, D2 to D31, D35 to D32, D40 to D33, D41 to D34, D42 to D35, D43 to D36, D44 to D37, D45 to D38, D46 to D39, D23 to D4, D47 to D40, D48 to D41, D49 to D42, D50 to D43, D51 to D44, D52 to D45, D3 to D46, D36 to D47, D53 to D48, D54 to D49, D24 to D5, D55 to D50, D56 to D51, D57 to D52, D58 to D53, D59 to D54, D60 to D55, D61 to D56, D62 to D57, D63 to D58, D65 to D59, D25 to D6, D4 to D60, D37 to D61, D26 to D7, D5 to D74, D38 to D75, D39 to D76, D27 to D8, D28 to D9, SW20 to SW1, SW29 to SW10, SW30 to SW11, SW31 to SW12, SW32 to SW13, SW33 to SW14, SW34 to SW15, SW1 to SW17, SW6 to SW18, SW7 to SW19, SW21 to SW2, SW8 to SW20, SW9 to SW21, SW10 to SW22, SW11 to SW23, SW12 to SW24, SW13 to SW25, SW14 to SW26, SW15 to SW27, SW16 to SW28, SW17 to SW29, SW22 to SW3, SW18 to SW30, SW19 to SW31, SW2 to SW32, SW35 to SW33, SW40 to SW34, SW41 to SW35, SW42 to SW36, SW43 to SW37, SW44 to SW38, SW45 to SW39, SW23 to SW4, SW46 to SW40, SW47 to SW41, SW48 to SW42, SW49 to SW43, SW50 to SW44, SW51 to SW45, SW52 to SW46, SW3 to SW47, SW36 to SW48, SW53 to SW49, SW24 to SW5, SW54 to SW50, SW55 to SW51, SW56 to SW52, SW57 to SW53, SW58 to SW54, SW59 to SW55, SW60 to SW56, SW61 to SW57, SW62 to SW58, SW63 to SW59, SW25 to SW6, SW65 to SW60, SW4 to SW61, SW37 to SW62, SW26 to SW7, SW5 to SW75, SW38 to SW76, SW39 to SW77, SW27 to SW8, SW28 to SW9
Connections:
- net COL3: now reaches SW4.1
- net COL3: now also A1.11 (GPIO8), SW20.1, SW35.1, SW50.1, SW64.1, SW78.1
- net ROW2: now reaches D45.1 (K)
- net ROW2: now also A1.2 (GPIO1), D31.1 (K), D32.1 (K), D33.1 (K), D34.1 (K), D35.1 (K), D36.1 (K), D37.1 (K), D38.1 (K), D39.1 (K), D40.1 (K), D41.1 (K), D42.1 (K), D43.1 (K), D44.1 (K)
- net ROW0: now reaches D6.1 (K)
- net ROW0: now also D1.1 (K), D10.1 (K), D11.1 (K), D12.1 (K), D13.1 (K), D14.1 (K), D15.1 (K), D2.1 (K), D3.1 (K), D4.1 (K), D5.1 (K), D7.1 (K), D8.1 (K), D9.1 (K)
- net COL5: now reaches SW37.1
- net COL5: now also A1.14 (GPIO10), SW22.1, SW52.1, SW6.1, SW66.1, SW80.1
- net COL6: now reaches SW53.1
- net COL6: now also A1.15 (GPIO11), SW23.1, SW38.1, SW7.1, SW67.1, SW81.1
- net ROW1: now reaches D19.1 (K)
- net ROW1: now also A1.1 (GPIO0), D16.1 (K), D17.1 (K), D18.1 (K), D20.1 (K), D21.1 (K), D22.1 (K), D23.1 (K), D24.1 (K), D25.1 (K), D26.1 (K), D27.1 (K), D28.1 (K), D29.1 (K), D30.1 (K)
- net COL14: now reaches SW60.1
- net COL14: now also A1.25 (GPIO19), SW15.1, SW31.1, SW46.1, SW74.1, SW88.1
- net COL0: now reaches SW17.1
- net COL0: now also A1.7 (GPIO5), SW1.1, SW32.1, SW47.1, SW61.1, SW75.1
- net COL1: now reaches SW76.1
- net COL1: now also A1.9 (GPIO6), SW18.1, SW2.1, SW33.1, SW48.1, SW62.1
- net ROW3: now reaches D57.1 (K)
- net ROW3: now also A1.4 (GPIO2), D46.1 (K), D47.1 (K), D48.1 (K), D49.1 (K), D50.1 (K), D51.1 (K), D52.1 (K), D53.1 (K), D54.1 (K), D55.1 (K), D56.1 (K), D58.1 (K), D59.1 (K)
- net COL8: now reaches SW55.1
- net COL8: now also A1.17 (GPIO13), SW25.1, SW40.1, SW9.1, SW69.1, SW83.1
- net COL7: now reaches SW39.1
- net COL7: now also A1.16 (GPIO12), SW24.1, SW54.1, SW8.1, SW68.1, SW82.1
- net COL4: now reaches SW5.1
- net COL4: now also A1.12 (GPIO9), SW21.1, SW36.1, SW51.1, SW65.1, SW79.1
- net COL9: now reaches SW10.1
- net COL9: now also A1.19 (GPIO14), SW26.1, SW41.1, SW56.1, SW70.1, SW84.1
- net ROW5: now reaches D74.1 (K)
- net ROW5: now also A1.6 (GPIO4), D75.1 (K), D76.1 (K), D77.1 (K), D78.1 (K), D79.1 (K), D80.1 (K), D81.1 (K), D82.1 (K), D83.1 (K), D84.1 (K), D85.1 (K), D86.1 (K), D87.1 (K)
- net ROW4: now reaches D61.1 (K)
- net ROW4: now also A1.5 (GPIO3), D60.1 (K), D62.1 (K), D63.1 (K), D64.1 (K), D65.1 (K), D66.1 (K), D67.1 (K), D68.1 (K), D69.1 (K), D70.1 (K), D71.1 (K), D72.1 (K), D73.1 (K)
- net COL11: now reaches SW12.1
- net COL11: now also A1.21 (GPIO16), SW28.1, SW43.1, SW58.1, SW72.1
- net COL10: now reaches SW11.1
- net COL10: now also A1.20 (GPIO15), SW27.1, SW42.1, SW57.1, SW71.1, SW85.1
- net COL12: now reaches SW29.1
- net COL12: now also A1.22 (GPIO17), SW13.1, SW44.1, SW86.1
- net COL2: now reaches SW19.1
- net COL2: now also A1.10 (GPIO7), SW3.1, SW34.1, SW49.1, SW77.1, SW63.1
- net COL13: now reaches SW14.1
- net COL13: now also A1.24 (GPIO18), SW30.1, SW45.1, SW59.1, SW73.1, SW87.1
- net GND: now reaches A1.13 (GND), A1.18 (GND), A1.23 (GND), A1.28 (GND), A1.3 (GND), A1.38 (GND), A1.8 (GND)
- net GND: now also SW16.C, SW16.S2, U1.1 (GND)
- net ROT0: now reaches A1.26 (GPIO20)
- net ROT0: now also SW16.S1
- net ROT1: now reaches A1.27 (GPIO21)
- net ROT1: now also SW16.A
- net ROT2: now reaches A1.29 (GPIO22)
- net ROT2: now also SW16.B
- net OLED2: now reaches A1.31 (GPIO26_ADC0)
- net OLED2: now also U1.4 (SDA)
- net OLED1: now reaches A1.32 (GPIO27_ADC1)
- net OLED1: now also U1.3 (SCL)
- net 3V3: now reaches A1.36 (3V3)
- net 3V3: now also U1.2 (VCC)
- new net: D67.2 (A), SW68.2
- new net: D80.2 (A), SW81.2
- new net: D82.2 (A), SW83.2
- new net: D85.2 (A), SW86.2
- new net: D65.2 (A), SW66.2
- new net: D71.2 (A), SW72.2
- new net: D84.2 (A), SW85.2
- new net: D62.2 (A), SW63.2
- new net: D77.2 (A), SW78.2
- new net: D64.2 (A), SW65.2
- new net: D86.2 (A), SW87.2
- new net: D69.2 (A), SW70.2
- new net: D66.2 (A), SW67.2
- new net: D79.2 (A), SW80.2
- new net: D72.2 (A), SW73.2
- new net: D83.2 (A), SW84.2
- new net: D81.2 (A), SW82.2
- new net: D70.2 (A), SW71.2
- new net: D63.2 (A), SW64.2
- new net: D78.2 (A), SW79.2
- new net: D68.2 (A), SW69.2
- new net: D73.2 (A), SW74.2
- new net: D87.2 (A), SW88.2
Other:
- moved on the sheet: A1, D32, D33, D34, D35, D36, D37, D38, D39, D40, D41, D42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
